Commit message: Feature: Add pluel blend 140 1

File: src/robots/community_robot_arm/urdf/community_robot_arm_slim.urdf (robot description, URDF)
Before this commit: robot complete_robotic_arm_assembly_with_dual_manipulator_140mm_shank, 35 links, 34 joints
Links:
- removed link 28BYJ_48 5V Stepper Motor
- removed link Parallel 2_0
- removed link Parallel 2_1
- removed link Parallel 2_2
- removed link gripperBase_by_ftobler
- removed link gripperFinger_by_ftobler
- removed link gripperFinger_by_ftobler_1
- removed link gripper_Finger_Washer _ myMOD
- removed link gripper_Finger_Washer _ myMOD_1
- removed link gripper_Fingers_Link_Wire
- removed link gripper_Fingers_Link_Wire_1
- removed link pleuel_bend_140_Mirrored
- removed link pleuel_bend_140_Mirrored_1
- removed link robot_belt_arm basering
- removed link robot_belt_arm endstop _ myMOD
- removed link robot_belt_arm gear_body
- removed link robot_belt_arm gear_body_1
- removed link robot_belt_arm leg
- removed link robot_belt_arm leg_1
- removed link robot_belt_arm leg_2
- removed link robot_belt_arm lever _ myMOD
- removed link robot_belt_arm main_body_v2 _  _ myMOD
- removed link robot_belt_arm rotategear _ myMOD
- removed link robot_belt_arm socket_v2
- removed link robot_belt_arm stabilizer _ Logigate
- removed link robot_belt_arm triplate
- added link 28byj_48_5v_stepper_motor, mass 1.29383e-05; visual mesh filename=package://community_robot_arm/meshes/28byj_48_5v_stepper_mo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 scale=1 1 1
- added link f624zz_97, mass 2.52711e-07; visual mesh filename=package://community_robot_arm/meshes/f624zz_97.stl scale=1 1 1
- added link gripper_finger_washer___mymod, mass 2.57418e-07; visual mesh filename=package://community_robot_arm/meshes/gripper_finger_washer_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 scale=1 1 1
- added link gripper_finger_washer___mymod_1, mass 2.57418e-07; visual mesh filename=package://community_robot_arm/meshes/gripper_finger_washer_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 scale=1 1 1
- added link gripper_fingers_link_wire, mass 5.2548e-08; visual mesh filename=package://community_robot_arm/meshes/gripper_fingers_link_w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 scale=1 1 1
- added link gripper_fingers_link_wire_1, mass 5.2548e-08; visual mesh filename=package://community_robot_arm/meshes/gripper_fingers_link_w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 scale=1 1 1
- added link gripperbase_by_ftobler, mass 1.98957e-05; visual mesh filename=package://community_robot_arm/meshes/gripperbase_by_ftobler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 scale=1 1 1
- added link gripperfinger_by_ftobler, mass 6.4034e-06; visual mesh filename=package://community_robot_arm/meshes/gripperfinger_by_ftobl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 scale=1 1 1
- added link gripperfinger_by_ftobler_1, mass 6.4034e-06; visual mesh filename=package://community_robot_arm/meshes/gripperfinger_by_ftobl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 scale=1 1 1
- added link pleuel_bend_140_mirrored, mass 8.88371e-06; visual mesh filename=package://community_robot_arm/meshes/pleuel_bend_140_mirror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 scale=1 1 1
- added link pleuel_bend_140_mirrored_1, mass 8.88371e-06; visual mesh filename=package://community_robot_arm/meshes/pleuel_bend_140_mirror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 scale=1 1 1
- added link robot_belt_arm_basering, mass 1.01419e-05; visual mesh filename=package://community_robot_arm/meshes/robot_belt_arm_baserin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 scale=1 1 1
- added link robot_belt_arm_endstop___mymod, mass 4.31512e-06; visual mesh filename=package://community_robot_arm/meshes/robot_belt_arm_endstop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 scale=1 1 1
- added link robot_belt_arm_gear_body, mass 1.12002e-05; visual mesh filename=package://community_robot_arm/meshes/robot_belt_arm_gear_bo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 scale=1 1 1
- added link robot_belt_arm_gear_body_1, mass 1.12002e-05; visual mesh filename=package://community_robot_arm/meshes/robot_belt_arm_gear_bo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 scale=1 1 1
- added link robot_belt_arm_leg, mass 1.42189e-05; visual mesh filename=package://community_robot_arm/meshes/robot_belt_arm_leg_2.s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 scale=1 1 1
- added link robot_belt_arm_leg_1, mass 1.42189e-05; visual mesh filename=package://community_robot_arm/meshes/robot_belt_arm_leg_2.s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 scale=1 1 1
- added link robot_belt_arm_leg_2, mass 1.42189e-05; visual mesh filename=package://community_robot_arm/meshes/robot_belt_arm_leg_2.s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 scale=1 1 1
- added link robot_belt_arm_lever___mymod, mass 1.00295e-05; visual mesh filename=package://community_robot_arm/meshes/robot_belt_arm_lever__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 scale=1 1 1
- added link robot_belt_arm_main_body_v2______mymod, mass 4.47417e-05; visual mesh filename=package://community_robot_arm/meshes/robot_belt_arm_main_bo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 scale=1 1 1
- added link robot_belt_arm_rotategear___mymod, mass 1.60564e-05; visual mesh filename=package://community_robot_arm/meshes/robot_belt_arm_rotateg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 scale=1 1 1
- added link robot_belt_arm_socket_v2, mass 4.17145e-05; visual mesh filename=package://community_robot_arm/meshes/robot_belt_arm_socket_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 scale=1 1 1
- added link robot_belt_arm_stabilizer___logigate, mass 2.08009e-06; visual mesh filename=package://community_robot_arm/meshes/robot_belt_arm_stabili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 scale=1 1 1
- added link robot_belt_arm_triplate, mass 7.1204e-06; visual mesh filename=package://community_robot_arm/meshes/robot_belt_arm_triplat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 scale=1 1 1
Joints:
- removed joint Fastened 1_0
- removed joint Fastened 2_0
- removed joint Fastened 3_0
- removed joint Fastened 4_0
- removed joint Fastened 5_0
- removed joint Final_Motor_fastened_joint_0
- removed joint Final_Motor_fastened_joint_1
- removed joint Final_Motor_fastened_joint_2
- removed joint Final_Motor_fastened_joint_3
- removed joint Final_Motor_fastened_joint_4
- removed joint Final_Motor_fastened_joint_5
- removed joint Final_Motor_fastened_joint_6
- removed joint Final_Motor_fastened_joint_7
- removed joint Parallel 2_3
- removed joint Parallel 2_4
- removed joint Parallel 2_5
- removed joint Parallel 2_6
- removed joint Revolute 10_0
- removed joint Revolute 11_0
- removed joint Revolute 12_0
- removed joint Revolute 13_0
- removed joint Revolute 14_0
- removed joint Revolute 15_0
- removed joint Revolute 16_0
- removed joint Revolute 18_0
- removed joint Revolute 19_0
- removed joint Revolute 1_0
- removed joint Revolute 21_0
- removed joint Revolute 2_0
- removed joint Revolute 4_0
- removed joint Revolute 6_0
- removed joint Revolute 8_0
- removed joint Revolute 9_0
- added joint fastened_1_0: type fixed, parent robot_belt_arm_basering, child robot_belt_arm_leg, origin xyz=0.0999887 -0.101005 -0.0632 rpy=0 -0 0, axis 1 0 0
- added joint fastened_2_0: type fixed, parent robot_belt_arm_basering, child robot_belt_arm_leg_1, origin xyz=0.151989 -0.0490051 -0.0632 rpy=0 -0 1.5708, axis 1 0 0
- added joint fastened_3_0: type fixed, parent robot_belt_arm_basering, child robot_belt_arm_leg_2, origin xyz=0.0999887 0.00299489 -0.0632 rpy=0 -0 3.14159, axis 1 0 0
- added joint fastened_4_0: type fixed, parent robot_belt_arm_leg_2, child robot_belt_arm_socket_v2, origin xyz=0 0.01834 0.036 rpy=0 -0 3.14159, axis 1 0 0
- added joint fastened_5_0: type fixed, parent robot_belt_arm_gear_body_1, child lower_shank_140, origin xyz=-2.77556e-17 0.0065 5.55112e-17 rpy=0 -1.5708 -6.2421e-16, axis 0 -1 0
- added joint fastened_6_0: type fixed, parent robot_belt_arm_main_body_v2______mymod, child robot_belt_arm_stabilizer___logigate, origin xyz=0.021 0.023 0.0345 rpy=3.14159 1.11575e-15 -6.95971e-15, axis -1 0 0
- added joint fastened_7_0: type fixed, parent robot_belt_arm_main_body_v2______mymod, child robot_belt_arm_endstop___mymod, origin xyz=-0.0225 0.023 0.0385 rpy=-3.98519e-16 -2.34135e-17 5.21805e-15, axis 1 0 0
- added joint final_motor_fastened_joint_0: type fixed, parent gripperbase_by_ftobler, child gripperfinger_by_ftobler_1, origin xyz=0.199541 -0.0467529 -0.195348 rpy=7.61135e-15 3.49775e-15 -3.14159, axis 0 0 1
- added joint final_motor_fastened_joint_1: type fixed, parent gripperbase_by_ftobler, child gripperfinger_by_ftobler, origin xyz=-0.145292 0.0466209 -0.195348 rpy=-2.51811e-16 5.27346e-16 3.81627e-16, axis 0 0 1
- added joint final_motor_fastened_joint_2: type fixed, parent gripper_fingers_link_wire, child gripper_fingers_link_wire_1, origin xyz=-0.00527287 0.0177687 9.99485e-13 rpy=-1.01688e-15 -6.15966e-16 -0.0134012, axis 0 0 1
- added joint final_motor_fastened_joint_3: type fixed, parent gripper_shaft, child 28byj_48_5v_stepper_motor, origin xyz=0.175273 -0.041981 0.204848 rpy=1.5708 -1.44329e-15 -0.348517, axis 0 0 1
- added joint final_motor_fastened_joint_4: type fixed, parent gripper_finger_washer___mymod_1, child gripper_finger_washer___mymod, origin xyz=-0.34748 -0.0935381 -4.71845e-16 rpy=1.59044e-15 -6.6229e-15 -3.14159, axis 0 0 1
- added joint final_motor_fastened_joint_5: type fixed, parent gripperfinger_by_ftobler, child gripper_finger_washer___mymod_1, origin xyz=0.350607 -0.0217646 0.189648 rpy=7.09546e-16 -5.31213e-14 -0.123995, axis 0 0 1
- added joint final_motor_fastened_joint_6: type fixed, parent 28byj_48_5v_stepper_motor, child gripper_fingers_link_wire, origin xyz=0.0307288 -0.205348 -0.158644 rpy=0 -1.5708 -1.57351, axis 0 0 1
- added joint final_motor_fastened_joint_7: type fixed, parent gripper_finger_washer___mymod, child gripper_shaft, origin xyz=-0.20806 0.129344 -0.189148 rpy=-9.76842e-15 1.25299e-15 -1.09828, axis 0 0 1
- added joint revolute_10_0: type continuous, parent robot_belt_arm_main_body_v2______mymod, child robot_belt_arm_gear_body, origin xyz=3.8384e-08 0.0135 0.064 rpy=0 -1.5708 3.14159, axis 0 1 0
- added joint revolute_11_0: type continuous, parent robot_belt_arm_gear_body, child robot_belt_arm_lever___mymod, origin xyz=2.77556e-17 0 6.93889e-18 rpy=4.3064e-16 -0.127314 -3.14159, axis 0 -1 0
- added joint revolute_12_0: type continuous, parent robot_belt_arm_lever___mymod, child pleuel_140, origin xyz=-0.035954 -0.008 -0.0175303 rpy=1.5708 -0.0168583 -7.47425e-15, axis 0 0 -1
- added joint revolute_13_0: type continuous, parent robot_belt_arm_triplate, child pleuel_bend_140, origin xyz=-0.03 -0.0095 0.012 rpy=1.89172e-14 1.29555 8.81648e-15, axis 0 1 0
- added joint revolute_15_0: type continuous, parent robot_belt_arm_triplate, child pleuel_bend_140_mirrored_1, origin xyz=0.015 -0.006 0.02 rpy=1.11265e-14 1.40074 -3.14159, axis 0 -1 0
- added joint revolute_16_0: type continuous, parent lower_shank_140, child upper_shank_140, origin xyz=-0.139911 0.0205 -0.00500004 rpy=-1.5708 -1.09096 -1.26261e-14, axis 0 0 1
- added joint revolute_17_0: type continuous, parent lower_shank_140, child triplate_dual, origin xyz=-0.139911 0.0275 -0.005 rpy=-3.14159 -1.06005 3.14159, axis 0 -1 0
- added joint revolute_18_0: type continuous, parent triplate_dual, child pleuel_bend_140_mirrored, origin xyz=-0.03 0.012 0.012 rpy=-1.00484e-14 1.29555 -5.92e-15, axis 0 -1 0
- added joint revolute_19_0: type continuous, parent triplate_dual, child pleuel_bend_140_1, origin xyz=0.015 0.0065 0.02 rpy=-2.27895e-14 1.40074 3.14159, axis 0 1 0
- added joint revolute_1_0: type continuous, parent robot_belt_arm_socket_v2, child robot_belt_arm_main_body_v2______mymod, origin xyz=6.93889e-18 -0.0336603 0.0257 rpy=2.09752e-16 -1.6689e-16 1.46153, axis 0 0 -1
- added joint revolute_21_0: type continuous, parent upper_shank_140, child manipulator_dual, origin xyz=0.14 -1.29296e-09 -0.015 rpy=1.5708 -1.9984e-15 -0.990552, axis 0 -1 0
- added joint revolute_22_0: type continuous, parent manipulator_dual, child gripperbase_by_ftobler, origin xyz=0.0269997 0.00750003 -0.001 rpy=9.19543e-17 -1.04873e-16 5.41189e-16, axis 0 0 -1
- added joint revolute_2_0: type continuous, parent robot_belt_arm_main_body_v2______mymod, child robot_belt_arm_rotategear___mymod, origin xyz=1.38778e-17 6.93889e-18 0 rpy=1.80866e-16 -2.08813e-16 -1.46153, axis 0 0 -1
- added joint revolute_3_0: type continuous, parent pleuel_bend_140, child f624zz_97, origin xyz=0.102411 -0.00500004 -0.0954576 rpy=1.5708 -0 -1.5708, axis -1 0 0
- added joint revolute_7_0: type continuous, parent lower_shank_140, child robot_belt_arm_triplate, origin xyz=-0.139911 -0.003 -0.005 rpy=-3.14159 -1.06005 3.14159, axis 0 1 0
- added joint revolute_9_0: type continuous, parent robot_belt_arm_main_body_v2______mymod, child robot_belt_arm_gear_body_1, origin xyz=3.8384e-08 -0.02 0.064 rpy=-3.14159 -0.510761 3.14159, axis 0 1 0
- joint fixed_node_to_root_joint_0: child robot_belt_arm basering -> robot_belt_arm_basering
