Commit message: Feature: Complete links

File: src/robots/community_robot_arm/urdf/community_robot_arm_slim.urdf (robot description, URDF)
Before this commit: robot complete_robotic_arm_assembly_with_dual_manipulator_140mm_shank, 33 links, 32 joints
Links:
- removed link f624zz_97
- added link f624zz_103, mass 2.52711e-07; visual mesh filename=package://community_robot_arm/meshes/f624zz_90.stl scale=1 1 1
- added link f624zz_14, mass 2.52711e-07; visual mesh filename=package://community_robot_arm/meshes/f624zz_90.stl scale=1 1 1
- added link f624zz_23, mass 2.52711e-07; visual mesh filename=package://community_robot_arm/meshes/f624zz_90.stl scale=1 1 1
- added link f624zz_34, mass 2.52711e-07; visual mesh filename=package://community_robot_arm/meshes/f624zz_90.stl scale=1 1 1
- added link f624zz_46, mass 2.52711e-07; visual mesh filename=package://community_robot_arm/meshes/f624zz_90.stl scale=1 1 1
- added link f624zz_5, mass 2.52711e-07; visual mesh filename=package://community_robot_arm/meshes/f624zz_90.stl scale=1 1 1
- added link f624zz_55, mass 2.52711e-07; visual mesh filename=package://community_robot_arm/meshes/f624zz_90.stl scale=1 1 1
- added link f624zz_73, mass 2.52711e-07; visual mesh filename=package://community_robot_arm/meshes/f624zz_90.stl scale=1 1 1
- added link f624zz_78, mass 2.52711e-07; visual mesh filename=package://community_robot_arm/meshes/f624zz_90.stl scale=1 1 1
- added link f624zz_90, mass 2.52711e-07; visual mesh filename=package://community_robot_arm/meshes/f624zz_90.stl scale=1 1 1
- added link f686zz_83, mass 2.83426e-07; visual mesh filename=package://community_robot_arm/meshes/f686zz_83.stl scale=1 1 1
- added link limit_switch, mass 4.37372e-07; visual mesh filename=package://community_robot_arm/meshes/limit_switch_2.stl scale=1 1 1
- added link limit_switch_2, mass 4.37372e-07; visual mesh filename=package://community_robot_arm/meshes/limit_switch_2.stl scale=1 1 1
- added link prevailing_torque_hex_flange_nut_am_am_m6_n_1, mass 5.54873e-07; visual mesh filename=package://community_robot_arm/meshes/prevailing_torque_hex_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 scale=1 1 1
- added link socket_button_head_cap_screw_am_b18_3_4m___3_x_0_5_x_6_sbhcs___n, mass 6.89009e-08; visual mesh filename=package://community_robot_arm/meshes/socket_button_head_cap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 scale=1 1 1
- added link socket_button_head_cap_screw_am_b18_3_4m___3_x_0_5_x_6_sbhcs___n_1, mass 6.89009e-08; visual mesh filename=package://community_robot_arm/meshes/socket_button_head_cap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 scale=1 1 1
- added link socket_button_head_cap_screw_am_b18_3_4m___3_x_0_5_x_8_sbhcs___n_1, mass 8.30381e-08; visual mesh filename=package://community_robot_arm/meshes/socket_button_head_cap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 scale=1 1 1
- added link socket_button_head_cap_screw_am_b18_3_4m___3_x_0_5_x_8_sbhcs___n_10, mass 8.30381e-08; visual mesh filename=package://community_robot_arm/meshes/socket_button_head_cap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 scale=1 1 1
- added link socket_button_head_cap_screw_am_b18_3_4m___3_x_0_5_x_8_sbhcs___n_13, mass 8.30381e-08; visual mesh filename=package://community_robot_arm/meshes/socket_button_head_cap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 scale=1 1 1
- added link socket_button_head_cap_screw_am_b18_3_4m___3_x_0_5_x_8_sbhcs___n_15, mass 8.30381e-08; visual mesh filename=package://community_robot_arm/meshes/socket_button_head_cap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 scale=1 1 1
- added link socket_button_head_cap_screw_am_b18_3_4m___3_x_0_5_x_8_sbhcs___n_17, mass 8.30381e-08; visual mesh filename=package://community_robot_arm/meshes/socket_button_head_cap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 scale=1 1 1
- added link socket_button_head_cap_screw_am_b18_3_4m___3_x_0_5_x_8_sbhcs___n_2, mass 8.30381e-08; visual mesh filename=package://community_robot_arm/meshes/socket_button_head_cap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 scale=1 1 1
- added link socket_button_head_cap_screw_am_b18_3_4m___3_x_0_5_x_8_sbhcs___n_3, mass 8.30381e-08; visual mesh filename=package://community_robot_arm/meshes/socket_button_head_cap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 scale=1 1 1
- added link socket_button_head_cap_screw_am_b18_3_4m___3_x_0_5_x_8_sbhcs___n_8, mass 8.30381e-08; visual mesh filename=package://community_robot_arm/meshes/socket_button_head_cap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 scale=1 1 1
- added link socket_button_head_cap_screw_am_b18_3_4m___4_x_0_7_x_20_sbhcs___n_4, mass 3.14324e-07; visual mesh filename=package://community_robot_arm/meshes/socket_button_head_cap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 scale=1 1 1
- added link socket_head_cap_screw_am_b18_3_1m___3_x_0_5_x_10_hex_shcs____10nhx_1, mass 1.32238e-07; visual mesh filename=package://community_robot_arm/meshes/socket_head_cap_screw_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 scale=1 1 1
- added link socket_head_cap_screw_am_b18_3_1m___3_x_0_5_x_10_hex_shcs____10nhx_4, mass 1.32238e-07; visual mesh filename=package://community_robot_arm/meshes/socket_head_cap_screw_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 scale=1 1 1
- added link socket_head_cap_screw_am_b18_3_1m___3_x_0_5_x_20_hex_shcs____20nhx, mass 2.02924e-07; visual mesh filename=package://community_robot_arm/meshes/socket_head_cap_screw_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 scale=1 1 1
- added link socket_head_cap_screw_am_b18_3_1m___3_x_0_5_x_20_hex_shcs____20nhx_1, mass 2.02924e-07; visual mesh filename=package://community_robot_arm/meshes/socket_head_cap_screw_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 scale=1 1 1
- added link socket_head_cap_screw_am_b18_3_1m___3_x_0_5_x_20_hex_shcs____20nhx_2, mass 2.02924e-07; visual mesh filename=package://community_robot_arm/meshes/socket_head_cap_screw_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 scale=1 1 1
- added link socket_head_cap_screw_am_b18_3_1m___3_x_0_5_x_20_hex_shcs____20nhx_3, mass 2.02924e-07; visual mesh filename=package://community_robot_arm/meshes/socket_head_cap_screw_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 scale=1 1 1
- added link socket_head_cap_screw_am_b18_3_1m___3_x_0_5_x_8_hex_shcs____8nhx, mass 1.18101e-07; visual mesh filename=package://community_robot_arm/meshes/socket_head_cap_screw_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 scale=1 1 1
- added link socket_head_cap_screw_am_b18_3_1m___3_x_0_5_x_8_hex_shcs____8nhx_1, mass 1.18101e-07; visual mesh filename=package://community_robot_arm/meshes/socket_head_cap_screw_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 scale=1 1 1
- added link socket_head_cap_screw_am_b18_3_1m___3_x_0_5_x_8_hex_shcs____8nhx_2, mass 1.18101e-07; visual mesh filename=package://community_robot_arm/meshes/socket_head_cap_screw_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 scale=1 1 1
- added link socket_head_cap_screw_am_b18_3_1m___3_x_0_5_x_8_hex_shcs____8nhx_3, mass 1.18101e-07; visual mesh filename=package://community_robot_arm/meshes/socket_head_cap_screw_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 scale=1 1 1
- added link socket_head_cap_screw_am_b18_3_1m___6_x_1_0_x_40_hex_shcs____24nhx, mass 1.51724e-06; visual mesh filename=package://community_robot_arm/meshes/socket_head_cap_screw_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 scale=1 1 1
Joints:
- removed joint revolute_17_0
- removed joint revolute_7_0
- added joint fastened_10_0: type fixed, parent 28byj_48_5v_stepper_motor, child socket_button_head_cap_screw_am_b18_3_4m___3_x_0_5_x_6_sbhcs___n, origin xyz=-0.0175 0.0008 0 rpy=-3.14159 1.93505e-15 -1.5708, axis 1 0 0
- added joint fastened_11_0: type fixed, parent robot_belt_arm_stabilizer___logigate, child socket_head_cap_screw_am_b18_3_1m___3_x_0_5_x_8_hex_shcs____8nhx, origin xyz=0.003 1.38778e-17 2.77556e-17 rpy=-3.14159 1.96753e-30 3.14159, axis 1 0 0
- added joint fastened_12_0: type fixed, parent robot_belt_arm_stabilizer___logigate, child socket_head_cap_screw_am_b18_3_1m___3_x_0_5_x_8_hex_shcs____8nhx_2, origin xyz=0.003 0.046 -2.77556e-17 rpy=-3.14159 1.96753e-30 3.14159, axis 1 0 0
- added joint fastened_13_0: type fixed, parent robot_belt_arm_stabilizer___logigate, child socket_head_cap_screw_am_b18_3_1m___3_x_0_5_x_8_hex_shcs____8nhx_1, origin xyz=0.003 2.77556e-17 0.01 rpy=-3.14159 1.96753e-30 3.14159, axis 1 0 0
- added joint fastened_14_0: type fixed, parent robot_belt_arm_stabilizer___logigate, child socket_head_cap_screw_am_b18_3_1m___3_x_0_5_x_8_hex_shcs____8nhx_3, origin xyz=0.003 0.046 0.01 rpy=-3.14159 1.96753e-30 3.14159, axis 1 0 0
- added joint fastened_15_0: type fixed, parent robot_belt_arm_endstop___mymod, child socket_button_head_cap_screw_am_b18_3_4m___3_x_0_5_x_8_sbhcs___n_2, origin xyz=-0.0035 -0.046 5.55112e-17 rpy=1.5708 1.65263e-16 1.12293e-16, axis 1 0 0
- added joint fastened_16_0: type fixed, parent robot_belt_arm_endstop___mymod, child socket_button_head_cap_screw_am_b18_3_4m___3_x_0_5_x_8_sbhcs___n_10, origin xyz=-0.0035 -0.046 -0.01 rpy=1.5708 1.65263e-16 1.12293e-16, axis 1 0 0
- added joint fastened_17_0: type fixed, parent robot_belt_arm_endstop___mymod, child socket_button_head_cap_screw_am_b18_3_4m___3_x_0_5_x_8_sbhcs___n_8, origin xyz=-0.0035 0 -0.01 rpy=1.5708 1.65263e-16 1.12293e-16, axis 1 0 0
- added joint fastened_18_0: type fixed, parent robot_belt_arm_endstop___mymod, child socket_button_head_cap_screw_am_b18_3_4m___3_x_0_5_x_8_sbhcs___n_1, origin xyz=-0.0035 0 2.77556e-17 rpy=1.5708 -6.06318e-15 -6.20479e-15, axis 1 0 0
- added joint fastened_19_0: type fixed, parent robot_belt_arm_main_body_v2______mymod, child socket_button_head_cap_screw_am_b18_3_4m___3_x_0_5_x_8_sbhcs___n_13, origin xyz=0.0135 0.0135 0.0045 rpy=0 1.5708 1.5708, axis 1 0 0
- added joint fastened_20_0: type fixed, parent robot_belt_arm_main_body_v2______mymod, child socket_button_head_cap_screw_am_b18_3_4m___3_x_0_5_x_8_sbhcs___n_15, origin xyz=0.0135 -0.0135 0.0045 rpy=0 1.5708 1.5708, axis 1 0 0
- added joint fastened_21_0: type fixed, parent robot_belt_arm_main_body_v2______mymod, child socket_button_head_cap_screw_am_b18_3_4m___3_x_0_5_x_8_sbhcs___n_3, origin xyz=-0.0135 -0.0135 0.0045 rpy=0 1.5708 1.5708, axis 1 0 0
- added joint fastened_22_0: type fixed, parent robot_belt_arm_main_body_v2______mymod, child socket_button_head_cap_screw_am_b18_3_4m___3_x_0_5_x_8_sbhcs___n_17, origin xyz=-0.0135 0.0135 0.0045 rpy=0 1.5708 1.5708, axis 1 0 0
- added joint fastened_23_0: type fixed, parent robot_belt_arm_gear_body_1, child socket_head_cap_screw_am_b18_3_1m___3_x_0_5_x_20_hex_shcs____20nhx_1, origin xyz=0.00999996 0.004 0 rpy=-1.88426e-17 6.21203e-17 1.5708, axis 1 0 0
- added joint fastened_24_0: type fixed, parent robot_belt_arm_gear_body_1, child socket_head_cap_screw_am_b18_3_1m___3_x_0_5_x_20_hex_shcs____20nhx_2, origin xyz=0 0.004 -0.01 rpy=-1.35122e-16 -1.0967e-16 1.5708, axis 1 0 0
- added joint fastened_25_0: type fixed, parent robot_belt_arm_gear_body_1, child socket_head_cap_screw_am_b18_3_1m___3_x_0_5_x_20_hex_shcs____20nhx, origin xyz=-0.01 0.004 1.38778e-17 rpy=-2.79844e-16 -8.78588e-17 1.5708, axis 1 0 0
- added joint fastened_26_0: type fixed, parent robot_belt_arm_gear_body_1, child socket_head_cap_screw_am_b18_3_1m___3_x_0_5_x_20_hex_shcs____20nhx_3, origin xyz=0 0.004 0.01 rpy=1.5708 -2.83107e-15 1.5708, axis 1 0 0
- added joint fastened_27_0: type fixed, parent robot_belt_arm_endstop___mymod, child limit_switch, origin xyz=-0.005 -0.019 -0.001488 rpy=0 -1.5708 4.71239, axis 0 1 0
- added joint fastened_28_0: type fixed, parent robot_belt_arm_endstop___mymod, child limit_switch_2, origin xyz=-0.0104652 -0.031 0.031735 rpy=-8.33744e-18 -3.92985e-17 2.77556e-17, axis 0 -1 0
- added joint fastened_30_0: type fixed, parent robot_belt_arm_socket_v2, child socket_head_cap_screw_am_b18_3_1m___3_x_0_5_x_10_hex_shcs____10nhx_4, origin xyz=-0.053 -0.0491602 0.005 rpy=0 1.5708 -0, axis 1 0 0
- added joint fastened_8_0: type fixed, parent manipulator_dual, child socket_button_head_cap_screw_am_b18_3_4m___4_x_0_7_x_20_sbhcs___n_4, origin xyz=0.0269997 0.00750003 -0.00700002 rpy=0 -1.5708 3.14159, axis 1 0 0
- added joint fastened_9_0: type fixed, parent 28byj_48_5v_stepper_motor, child socket_button_head_cap_screw_am_b18_3_4m___3_x_0_5_x_6_sbhcs___n_1, origin xyz=0.0175 0.0008 0 rpy=-3.14159 4.0268e-16 -1.5708, axis 1 0 0
- added joint revolute_14_0: type continuous, parent pleuel_bend_140_mirrored_1, child f624zz_103, origin xyz=0.102411 0.00500004 -0.0954576 rpy=1.5708 -1.12688e-14 1.5708, axis -1 0 0
- added joint revolute_24_0: type continuous, parent robot_belt_arm_triplate, child f686zz_83, origin xyz=0.03 0.0089 -0.012 rpy=-0.377454 4.77396e-15 -1.5708, axis -1 0 0
- added joint revolute_25_0: type continuous, parent pleuel_140, child f624zz_23, origin xyz=-0.11402 0.0812835 0.001 rpy=0 1.5708 -3.56578e-06, axis -1 0 0
- added joint revolute_26_0: type continuous, parent pleuel_bend_140_mirrored_1, child f624zz_90, origin xyz=-5.55112e-17 0.00500004 -1.04083e-17 rpy=-1.5708 -2.22045e-16 1.5708, axis -1 0 0
- added joint revolute_27_0: type continuous, parent pleuel_bend_140_1, child f624zz_34, origin xyz=0 -0.00500004 -1.38778e-17 rpy=1.5708 4.996e-16 -1.5708, axis -1 0 0
- added joint revolute_28_0: type continuous, parent pleuel_bend_140_mirrored, child f624zz_5, origin xyz=-0.102411 0.00500004 0.0954576 rpy=-1.84603 -5.55112e-17 1.5708, axis -1 0 0
- added joint revolute_29_0: type continuous, parent pleuel_bend_140, child f624zz_46, origin xyz=-0.102411 -0.00500004 0.0954576 rpy=1.84603 -4.4964e-15 -1.5708, axis -1 0 0
- added joint revolute_30_0: type continuous, parent robot_belt_arm_main_body_v2______mymod, child prevailing_torque_hex_flange_nut_am_am_m6_n_1, origin xyz=3.8384e-08 0.026 0.064 rpy=-1.5708 5.88418e-15 5.85208e-15, axis 0 0 -1
- added joint revolute_31_0: type continuous, parent robot_belt_arm_main_body_v2______mymod, child pleuel_bend_140_mirrored, origin xyz=-0.03 0.026 0.076 rpy=-3.14159 1.44879 -3.14159, axis 0 -1 0
- added joint revolute_32_0: type continuous, parent robot_belt_arm_main_body_v2______mymod, child pleuel_bend_140, origin xyz=-0.03 -0.026 0.076 rpy=-3.14159 1.44879 -3.14159, axis 0 1 0
- added joint revolute_33_0: type continuous, parent robot_belt_arm_socket_v2, child socket_head_cap_screw_am_b18_3_1m___3_x_0_5_x_10_hex_shcs____10nhx_1, origin xyz=-0.053 -0.0181602 0.005 rpy=0 1.5708 -0, axis 1 0 0
- added joint revolute_4_0: type continuous, parent pleuel_bend_140_mirrored, child f624zz_78, origin xyz=2.77556e-17 0.00500004 4.16334e-17 rpy=-1.84603 7.21645e-16 1.5708, axis -1 0 0
- added joint revolute_5_0: type continuous, parent manipulator_dual, child socket_head_cap_screw_am_b18_3_1m___6_x_1_0_x_40_hex_shcs____24nhx, origin xyz=-2.77556e-17 -0.007 0 rpy=-8.87308e-07 1.56423e-15 1.5708, axis 1 0 0
- added joint revolute_6_0: type continuous, parent pleuel_140, child f624zz_14, origin xyz=-1.94289e-16 5.55112e-17 0.005 rpy=0 -1.5708 3.14159, axis -1 0 0
- added joint revolute_8_0: type continuous, parent pleuel_bend_140_1, child f624zz_73, origin xyz=0.102411 -0.00500004 -0.0954576 rpy=-1.09686 -1.52101e-14 -1.5708, axis -1 0 0
- joint fastened_4_0: origin xyz=0 0.01834 0.036 rpy=0 -0 3.14159 -> xyz=-6.93889e-18 0.01834 0.036 rpy=0 -0 3.14159
- joint fastened_5_0: origin xyz=-2.77556e-17 0.0065 5.55112e-17 rpy=0 -1.5708 -6.2421e-16 -> xyz=-2.77556e-17 0.0065 4.16334e-17 rpy=0 -1.5708 6.16777e-16
- joint fastened_6_0: origin xyz=0.021 0.023 0.0345 rpy=3.14159 1.11575e-15 -6.95971e-15 -> xyz=0.021 0.023 0.0345 rpy=3.14159 1.11575e-15 6.10623e-15
- joint fastened_7_0: origin xyz=-0.0225 0.023 0.0385 rpy=-3.98519e-16 -2.34135e-17 5.21805e-15 -> xyz=-0.0225 0.023 0.0385 rpy=-3.98519e-16 -2.34135e-17 -3.38618e-15
- joint final_motor_fastened_joint_0: origin xyz=0.199541 -0.0467529 -0.195348 rpy=7.61135e-15 3.49775e-15 -3.14159 -> xyz=0.199541 -0.0467529 -0.195348 rpy=7.61356e-15 3.49877e-15 -3.14159
- joint final_motor_fastened_joint_1: origin xyz=-0.145292 0.0466209 -0.195348 rpy=-2.51811e-16 5.27346e-16 3.81627e-16 -> xyz=-0.145292 0.0466209 -0.195348 rpy=-2.52509e-16 5.33644e-16 -5.55126e-17
- joint final_motor_fastened_joint_2: origin xyz=-0.00527287 0.0177687 9.99485e-13 rpy=-1.01688e-15 -6.15966e-16 -0.0134012 -> xyz=-0.00527287 0.0177687 9.9951e-13 rpy=-1.01871e-15 -6.12848e-16 -0.0134012
- joint final_motor_fastened_joint_3: origin xyz=0.175273 -0.041981 0.204848 rpy=1.5708 -1.44329e-15 -0.348517 -> xyz=0.175273 -0.041981 0.204848 rpy=1.5708 -4.16334e-16 -0.348517
- joint final_motor_fastened_joint_4: origin xyz=-0.34748 -0.0935381 -4.71845e-16 rpy=1.59044e-15 -6.6229e-15 -3.14159 -> xyz=-0.34748 -0.0935381 -8.32667e-16 rpy=1.586e-15 -6.62775e-15 -3.14159
- joint final_motor_fastened_joint_5: origin xyz=0.350607 -0.0217646 0.189648 rpy=7.09546e-16 -5.31213e-14 -0.123995 -> xyz=0.350607 -0.0217646 0.189648 rpy=7.06873e-16 -5.31245e-14 -0.123995
- joint final_motor_fastened_joint_7: origin xyz=-0.20806 0.129344 -0.189148 rpy=-9.76842e-15 1.25299e-15 -1.09828 -> xyz=-0.20806 0.129344 -0.189148 rpy=-9.77073e-15 1.25527e-15 -1.09828
- joint revolute_10_0: origin xyz=3.8384e-08 0.0135 0.064 rpy=0 -1.5708 3.14159 -> xyz=3.8384e-08 0.0135 0.064 rpy=3.14159 0.206001 2.87083e-15
- joint revolute_11_0: origin xyz=2.77556e-17 0 6.93889e-18 rpy=4.3064e-16 -0.127314 -3.14159 -> xyz=5.55112e-17 -1.38778e-17 -2.77556e-17 rpy=-3.14159 -1.40802 -3.09284e-14
- joint revolute_12_0: origin xyz=-0.035954 -0.008 -0.0175303 rpy=1.5708 -0.0168583 -7.47425e-15 -> xyz=-0.035954 -0.008 -0.0175303 rpy=1.5708 0.209788 6.52688e-16
- joint revolute_13_0: child pleuel_bend_140 -> robot_belt_arm_triplate; origin xyz=-0.03 -0.0095 0.012 rpy=1.89172e-14 1.29555 8.81648e-15 -> xyz=-0.102411 1.16229e-09 0.0954576 rpy=-3.14159 -1.44881 3.14159; parent robot_belt_arm_triplate -> pleuel_bend_140
- joint revolute_15_0: origin xyz=0.015 -0.006 0.02 rpy=1.11265e-14 1.40074 -3.14159 -> xyz=0.045 0.0035 0.008 rpy=4.88698e-16 1.23027 3.14159
- joint revolute_16_0: origin xyz=-0.139911 0.0205 -0.00500004 rpy=-1.5708 -1.09096 -1.26261e-14 -> xyz=-0.139911 0.0205 -0.005 rpy=-1.5708 -1.31772 -2.26142e-14
- joint revolute_18_0: child pleuel_bend_140_mirrored -> triplate_dual; origin xyz=-0.03 0.012 0.012 rpy=-1.00484e-14 1.29555 -5.92e-15 -> xyz=-0.102411 -1.11022e-16 0.0954576 rpy=3.14159 -1.44881 -3.14159; parent triplate_dual -> pleuel_bend_140_mirrored
- joint revolute_19_0: origin xyz=0.015 0.0065 0.02 rpy=-2.27895e-14 1.40074 3.14159 -> xyz=0.045 -0.0035 0.008 rpy=0 1.23027 -3.14159
- joint revolute_1_0: origin xyz=6.93889e-18 -0.0336603 0.0257 rpy=2.09752e-16 -1.6689e-16 1.46153 -> xyz=-2.08167e-17 -0.0336603 0.0257 rpy=1.90568e-16 1.59644e-16 -1.27729
- joint revolute_21_0: origin xyz=0.14 -1.29296e-09 -0.015 rpy=1.5708 -1.9984e-15 -0.990552 -> xyz=0.14 -1.29294e-09 -0.015 rpy=1.5708 -7.21645e-16 -1.16102
- joint revolute_22_0: origin xyz=0.0269997 0.00750003 -0.001 rpy=9.19543e-17 -1.04873e-16 5.41189e-16 -> xyz=0.0269997 0.00750003 -0.001 rpy=1.93138e-15 -4.34816e-16 2.80332e-15
- joint revolute_2_0: origin xyz=1.38778e-17 6.93889e-18 0 rpy=1.80866e-16 -2.08813e-16 -1.46153 -> xyz=3.81639e-17 1.38778e-17 0 rpy=-1.87643e-15 1.85486e-16 2.84045
- joint revolute_3_0: child f624zz_97 -> f624zz_55; origin xyz=0.102411 -0.00500004 -0.0954576 rpy=1.5708 -0 -1.5708 -> xyz=-5.55112e-17 -0.00500004 1.38778e-17 rpy=1.84603 -5.05151e-15 -1.5708
- joint revolute_9_0: origin xyz=3.8384e-08 -0.02 0.064 rpy=-3.14159 -0.510761 3.14159 -> xyz=-4.83882e-08 -0.02 0.064 rpy=-3.14159 -0.908 3.14159

Commit message: Feature: Set origin

File: src/robots/community_robot_arm/urdf/community_robot_arm_slim.urdf (robot description, URDF)
Before this commit: robot complete_robotic_arm_assembly_with_dual_manipulator_140mm_shank, 68 links, 67 joints
Joints:
- joint fixed_node_to_root_joint_0: origin xyz=-0.0604648 0.0900997 0.153201 rpy=0 -0 0 -> xyz=-0.101239 0.049005 0.0677 rpy=0 0 0
