Commit message: Feature: Adjust again

File: src/robots/community_robot_arm/urdf/community_robot_arm_slim.urdf (robot description, URDF)
Before this commit: robot complete_robotic_arm_assembly_with_dual_manipulator_140mm_shank, 68 links, 67 joints
Links:
- added link hex_nut_style_1_am_b18_2_4_1m___hex_nut__style_1___m2_5_x_0_45___d_n_1, mass 3.61428e-08; visual mesh filename=package://community_robot_arm/meshes/hex_nut_style_1_am_b18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 scale=1 1 1
- added link hex_nut_style_1_am_b18_2_4_1m___hex_nut__style_1___m2_5_x_0_45___d_n_2, mass 3.61428e-08; visual mesh filename=package://community_robot_arm/meshes/hex_nut_style_1_am_b18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 scale=1 1 1
- added link hex_nut_style_1_am_b18_2_4_1m___hex_nut__style_1___m2_5_x_0_45___d_n_3, mass 3.61428e-08; visual mesh filename=package://community_robot_arm/meshes/hex_nut_style_1_am_b18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 scale=1 1 1
- added link hex_nut_style_1_am_b18_2_4_1m___hex_nut__style_1___m2_5_x_0_45___d_n_5, mass 3.61428e-08; visual mesh filename=package://community_robot_arm/meshes/hex_nut_style_1_am_b18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 scale=1 1 1
- added link limit_switch_1, mass 4.37372e-07; visual mesh filename=package://community_robot_arm/meshes/limit_switch_2.stl scale=1 1 1
- added link parallel_4_0
- added link parallel_4_1
- added link parallel_4_2
- added link socket_button_head_cap_screw_am_b18_3_4m___3_x_0_5_x_8_sbhcs___n, mass 8.30381e-08; visual mesh filename=package://community_robot_arm/meshes/socket_button_head_cap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 scale=1 1 1
- added link socket_button_head_cap_screw_am_b18_3_4m___3_x_0_5_x_8_sbhcs___n_11, mass 8.30381e-08; visual mesh filename=package://community_robot_arm/meshes/socket_button_head_cap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 scale=1 1 1
- added link socket_button_head_cap_screw_am_b18_3_4m___3_x_0_5_x_8_sbhcs___n_12, mass 8.30381e-08; visual mesh filename=package://community_robot_arm/meshes/socket_button_head_cap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 scale=1 1 1
- added link socket_button_head_cap_screw_am_b18_3_4m___3_x_0_5_x_8_sbhcs___n_14, mass 8.30381e-08; visual mesh filename=package://community_robot_arm/meshes/socket_button_head_cap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 scale=1 1 1
- added link socket_button_head_cap_screw_am_b18_3_4m___3_x_0_5_x_8_sbhcs___n_16, mass 8.30381e-08; visual mesh filename=package://community_robot_arm/meshes/socket_button_head_cap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 scale=1 1 1
- added link socket_button_head_cap_screw_am_b18_3_4m___3_x_0_5_x_8_sbhcs___n_4, mass 8.30381e-08; visual mesh filename=package://community_robot_arm/meshes/socket_button_head_cap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 scale=1 1 1
- added link socket_button_head_cap_screw_am_b18_3_4m___3_x_0_5_x_8_sbhcs___n_5, mass 8.30381e-08; visual mesh filename=package://community_robot_arm/meshes/socket_button_head_cap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 scale=1 1 1
- added link socket_button_head_cap_screw_am_b18_3_4m___3_x_0_5_x_8_sbhcs___n_6, mass 8.30381e-08; visual mesh filename=package://community_robot_arm/meshes/socket_button_head_cap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 scale=1 1 1
- added link socket_button_head_cap_screw_am_b18_3_4m___3_x_0_5_x_8_sbhcs___n_7, mass 8.30381e-08; visual mesh filename=package://community_robot_arm/meshes/socket_button_head_cap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 scale=1 1 1
- added link socket_button_head_cap_screw_am_b18_3_4m___3_x_0_5_x_8_sbhcs___n_9, mass 8.30381e-08; visual mesh filename=package://community_robot_arm/meshes/socket_button_head_cap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 scale=1 1 1
- added link socket_head_cap_screw_am_b18_3_1m___2_5_x_0_45_x_10_hex_shcs____10nhx, mass 8.35744e-08; visual mesh filename=package://community_robot_arm/meshes/socket_head_cap_screw_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 scale=1 1 1
- added link socket_head_cap_screw_am_b18_3_1m___2_5_x_0_45_x_10_hex_shcs____10nhx_2, mass 8.35744e-08; visual mesh filename=package://community_robot_arm/meshes/socket_head_cap_screw_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 scale=1 1 1
- added link socket_head_cap_screw_am_b18_3_1m___2_5_x_0_45_x_10_hex_shcs____10nhx_3, mass 8.35744e-08; visual mesh filename=package://community_robot_arm/meshes/socket_head_cap_screw_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 scale=1 1 1
- added link socket_head_cap_screw_am_b18_3_1m___2_5_x_0_45_x_10_hex_shcs____10nhx_4, mass 8.35744e-08; visual mesh filename=package://community_robot_arm/meshes/socket_head_cap_screw_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 scale=1 1 1
- added link socket_head_cap_screw_am_b18_3_1m___3_x_0_5_x_10_hex_shcs____10nhx, mass 1.32238e-07; visual mesh filename=package://community_robot_arm/meshes/socket_head_cap_screw_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 scale=1 1 1
- added link socket_head_cap_screw_am_b18_3_1m___3_x_0_5_x_10_hex_shcs____10nhx_2, mass 1.32238e-07; visual mesh filename=package://community_robot_arm/meshes/socket_head_cap_screw_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 scale=1 1 1
- added link socket_head_cap_screw_am_b18_3_1m___3_x_0_5_x_10_hex_shcs____10nhx_3, mass 1.32238e-07; visual mesh filename=package://community_robot_arm/meshes/socket_head_cap_screw_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 scale=1 1 1
- added link socket_head_cap_screw_am_b18_3_1m___3_x_0_5_x_10_hex_shcs____10nhx_5, mass 1.32238e-07; visual mesh filename=package://community_robot_arm/meshes/socket_head_cap_screw_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 scale=1 1 1
- added link socket_head_cap_screw_am_b18_3_1m___3_x_0_5_x_10_hex_shcs____10nhx_6, mass 1.32238e-07; visual mesh filename=package://community_robot_arm/meshes/socket_head_cap_screw_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 scale=1 1 1
- added link socket_head_cap_screw_am_b18_3_1m___3_x_0_5_x_10_hex_shcs____10nhx_7, mass 1.32238e-07; visual mesh filename=package://community_robot_arm/meshes/socket_head_cap_screw_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 scale=1 1 1
Joints:
- removed joint revolute_21_0
- added joint fastened_31_0: type fixed, parent robot_belt_arm_main_body_v2______mymod, child socket_button_head_cap_screw_am_b18_3_4m___3_x_0_5_x_8_sbhcs___n_4, origin xyz=-0.0155 -0.022 0.0425 rpy=3.11173e-31 2.0095e-31 -1.5708, axis 1 0 0
- added joint fastened_32_0: type fixed, parent robot_belt_arm_main_body_v2______mymod, child socket_button_head_cap_screw_am_b18_3_4m___3_x_0_5_x_8_sbhcs___n_9, origin xyz=0.0155 -0.022 0.0425 rpy=9.89967e-31 2.12041e-31 -1.5708, axis 1 0 0
- added joint fastened_33_0: type fixed, parent robot_belt_arm_main_body_v2______mymod, child socket_button_head_cap_screw_am_b18_3_4m___3_x_0_5_x_8_sbhcs___n_6, origin xyz=-0.0155 -0.022 0.0115 rpy=-3.04483e-16 -5.16486e-16 -1.5708, axis 1 0 0
- added joint fastened_34_0: type fixed, parent robot_belt_arm_main_body_v2______mymod, child socket_button_head_cap_screw_am_b18_3_4m___3_x_0_5_x_8_sbhcs___n_12, origin xyz=0.0155 0.02 0.0425 rpy=-3.14159 -4.21932e-16 1.5708, axis 1 0 0
- added joint fastened_35_0: type fixed, parent robot_belt_arm_main_body_v2______mymod, child socket_button_head_cap_screw_am_b18_3_4m___3_x_0_5_x_8_sbhcs___n_7, origin xyz=-0.0155 0.022 0.0425 rpy=8.78734e-32 1.07211e-32 1.5708, axis 1 0 0
- added joint fastened_36_0: type fixed, parent robot_belt_arm_main_body_v2______mymod, child socket_button_head_cap_screw_am_b18_3_4m___3_x_0_5_x_8_sbhcs___n_14, origin xyz=0.0155 0.022 0.0115 rpy=2.04623e-30 3.82837e-31 1.5708, axis 1 0 0
- added joint fastened_37_0: type fixed, parent robot_belt_arm_main_body_v2______mymod, child socket_button_head_cap_screw_am_b18_3_4m___3_x_0_5_x_8_sbhcs___n, origin xyz=-0.0155 0.022 0.0115 rpy=1.82277e-30 2.5794e-31 1.5708, axis 1 0 0
- added joint fastened_38_0: type fixed, parent robot_belt_arm_main_body_v2______mymod, child socket_button_head_cap_screw_am_b18_3_4m___3_x_0_5_x_8_sbhcs___n_11, origin xyz=0.0155 -0.022 0.0115 rpy=3.14159 -3.75105e-16 -1.5708, axis 1 0 0
- added joint fastened_39_0: type fixed, parent robot_belt_arm_endstop___mymod, child socket_head_cap_screw_am_b18_3_1m___2_5_x_0_45_x_10_hex_shcs____10nhx_2, origin xyz=-0.0037 -0.019 -0.001488 rpy=1.5708 -6.22641e-15 -6.31911e-15, axis 1 0 0
- added joint fastened_40_0: type fixed, parent robot_belt_arm_endstop___mymod, child socket_head_cap_screw_am_b18_3_1m___2_5_x_0_45_x_10_hex_shcs____10nhx_3, origin xyz=-0.0037 -0.0255 -0.001488 rpy=1.5708 2.498e-16 2.31645e-16, axis 1 0 0
- added joint fastened_41_0: type fixed, parent robot_belt_arm_endstop___mymod, child socket_head_cap_screw_am_b18_3_1m___2_5_x_0_45_x_10_hex_shcs____10nhx_4, origin xyz=-0.00586899 -0.033 0.0271388 rpy=6.47909e-23 3.75144e-23 1.5708, axis 1 0 0
- added joint fastened_42_0: type fixed, parent robot_belt_arm_endstop___mymod, child socket_head_cap_screw_am_b18_3_1m___2_5_x_0_45_x_10_hex_shcs____10nhx, origin xyz=-0.0104652 -0.033 0.031735 rpy=6.47909e-23 3.75144e-23 1.5708, axis 1 0 0
- added joint fastened_43_0: type fixed, parent socket_head_cap_screw_am_b18_3_1m___2_5_x_0_45_x_10_hex_shcs____10nhx_3, child hex_nut_style_1_am_b18_2_4_1m___hex_nut__style_1___m2_5_x_0_45___d_n_5, origin xyz=0.0097465 -2.77556e-17 -5.20417e-18 rpy=0 1.5708 4.07471e-17, axis 0 0 -1
- added joint fastened_44_0: type fixed, parent socket_head_cap_screw_am_b18_3_1m___2_5_x_0_45_x_10_hex_shcs____10nhx_2, child hex_nut_style_1_am_b18_2_4_1m___hex_nut__style_1___m2_5_x_0_45___d_n_3, origin xyz=0.0097465 -5.55112e-17 0 rpy=0 -1.5708 -3.61459e-30, axis 0 0 -1
- added joint fastened_45_0: type fixed, parent robot_belt_arm_socket_v2, child socket_head_cap_screw_am_b18_3_1m___3_x_0_5_x_10_hex_shcs____10nhx_6, origin xyz=-0.022 -0.0181602 0.005 rpy=0 1.5708 -0, axis 1 0 0
- added joint fastened_46_0: type fixed, parent robot_belt_arm_socket_v2, child socket_head_cap_screw_am_b18_3_1m___3_x_0_5_x_10_hex_shcs____10nhx, origin xyz=-0.022 -0.0491602 0.005 rpy=0 1.5708 -0, axis 1 0 0
- added joint fastened_47_0: type fixed, parent socket_head_cap_screw_am_b18_3_1m___2_5_x_0_45_x_10_hex_shcs____10nhx, child hex_nut_style_1_am_b18_2_4_1m___hex_nut__style_1___m2_5_x_0_45___d_n_1, origin xyz=0.0097465 3.46945e-18 -2.77556e-17 rpy=0 -1.5708 3.14159, axis 0 0 1
- added joint fastened_48_0: type fixed, parent socket_head_cap_screw_am_b18_3_1m___2_5_x_0_45_x_10_hex_shcs____10nhx_4, child hex_nut_style_1_am_b18_2_4_1m___hex_nut__style_1___m2_5_x_0_45___d_n_2, origin xyz=0.0097465 -3.46945e-18 -2.77556e-17 rpy=0 -1.5708 3.14159, axis 0 0 -1
- added joint fastened_49_0: type fixed, parent gripper_finger_washer___mymod, child socket_button_head_cap_screw_am_b18_3_4m___3_x_0_5_x_8_sbhcs___n_5, origin xyz=-0.174416 -0.0251722 2.77556e-17 rpy=0 -1.5708 3.14159, axis 1 0 0
- added joint fastened_50_0: type fixed, parent gripper_finger_washer___mymod_1, child socket_button_head_cap_screw_am_b18_3_4m___3_x_0_5_x_8_sbhcs___n_16, origin xyz=-0.174416 -0.0251722 -2.77556e-17 rpy=0 -1.5708 4.38178e-17, axis 1 0 0
- added joint parallel_4_3: type prismatic, parent robot_belt_arm_main_body_v2______mymod, child parallel_4_2, origin xyz=-0.02115 -0.03151 0.027 rpy=1.5708 -6.69813e-15 3.14159, axis 0 1 0, limit lower=-10000 upper=10000 effort=1 velocity=1
- added joint parallel_4_4: type prismatic, parent parallel_4_2, child parallel_4_1, origin xyz=0 0 0 rpy=0 -0 0, axis 0 0 1, limit lower=-10000 upper=10000 effort=1 velocity=1
- added joint parallel_4_5: type prismatic, parent parallel_4_1, child parallel_4_0, origin xyz=0 0 0 rpy=0 -0 0, axis 1 0 0, limit lower=-10000 upper=10000 effort=1 velocity=1
- added joint revolute_23_0: type continuous, parent pleuel_bend_140_mirrored_1, child manipulator_dual, origin xyz=0.102411 -1.11022e-16 -0.0954576 rpy=-3.14159 1.43823 1.50858e-14, axis 0 1 0
- added joint revolute_34_0: type continuous, parent robot_belt_arm_endstop___mymod, child limit_switch_2, origin xyz=-0.0104652 -0.031 0.031735 rpy=-3.28385e-15 -0.785398 8.31403e-15, axis 0 -1 0
- added joint revolute_38_0: type continuous, parent robot_belt_arm_gear_body, child socket_head_cap_screw_am_b18_3_1m___3_x_0_5_x_10_hex_shcs____10nhx_5, origin xyz=-1.82146e-17 -0.0025 -0.01 rpy=3.44926e-14 1.99844e-15 1.5708, axis 1 0 0
- added joint revolute_39_0: type continuous, parent robot_belt_arm_gear_body, child socket_head_cap_screw_am_b18_3_1m___3_x_0_5_x_10_hex_shcs____10nhx_3, origin xyz=-4.33681e-18 -0.0025 0.01 rpy=3.44926e-14 1.99844e-15 1.5708, axis 1 0 0
- added joint revolute_40_0: type continuous, parent robot_belt_arm_gear_body, child socket_head_cap_screw_am_b18_3_1m___3_x_0_5_x_10_hex_shcs____10nhx_2, origin xyz=-0.01 -0.0025 -2.77556e-17 rpy=-1.5708 -1.11022e-15 1.5708, axis 1 0 0
- added joint revolute_41_0: type continuous, parent robot_belt_arm_gear_body, child socket_head_cap_screw_am_b18_3_1m___3_x_0_5_x_10_hex_shcs____10nhx_7, origin xyz=0.00999996 -0.0025 -2.77556e-17 rpy=3.44926e-14 1.99844e-15 1.5708, axis 1 0 0
- joint fastened_10_0: origin xyz=-0.0175 0.0008 0 rpy=-3.14159 1.93505e-15 -1.5708 -> xyz=-0.0175 0.0008 -5.55112e-17 rpy=3.14159 1.22954e-15 -1.5708
- joint fastened_11_0: origin xyz=0.003 1.38778e-17 2.77556e-17 rpy=-3.14159 1.96753e-30 3.14159 -> xyz=0.003 0 -2.77556e-17 rpy=-3.14159 -1.02305e-22 -3.14159
- joint fastened_12_0: origin xyz=0.003 0.046 -2.77556e-17 rpy=-3.14159 1.96753e-30 3.14159 -> xyz=0.003 0.046 0 rpy=-3.14159 -1.02305e-22 -3.14159
- joint fastened_13_0: origin xyz=0.003 2.77556e-17 0.01 rpy=-3.14159 1.96753e-30 3.14159 -> xyz=0.003 -1.38778e-17 0.01 rpy=-3.14159 -1.02305e-22 -3.14159
- joint fastened_14_0: origin xyz=0.003 0.046 0.01 rpy=-3.14159 1.96753e-30 3.14159 -> xyz=0.003 0.046 0.01 rpy=-3.14159 -1.02305e-22 -3.14159
- joint fastened_15_0: origin xyz=-0.0035 -0.046 5.55112e-17 rpy=1.5708 1.65263e-16 1.12293e-16 -> xyz=-0.0035 -0.046 -5.55112e-17 rpy=1.5708 -1.67804e-16 -1.09752e-16
- joint fastened_16_0: origin xyz=-0.0035 -0.046 -0.01 rpy=1.5708 1.65263e-16 1.12293e-16 -> xyz=-0.0035 -0.046 -0.01 rpy=1.5708 -1.67804e-16 -1.09752e-16
- joint fastened_17_0: origin xyz=-0.0035 0 -0.01 rpy=1.5708 1.65263e-16 1.12293e-16 -> xyz=-0.0035 6.93889e-18 -0.01 rpy=1.5708 -1.67804e-16 -1.09752e-16
- joint fastened_18_0: origin xyz=-0.0035 0 2.77556e-17 rpy=1.5708 -6.06318e-15 -6.20479e-15 -> xyz=-0.0035 1.38778e-17 -8.32667e-17 rpy=1.5708 -6.1742e-15 -6.37132e-15
- joint fastened_23_0: origin xyz=0.00999996 0.004 0 rpy=-1.88426e-17 6.21203e-17 1.5708 -> xyz=0.00999996 0.004 -5.55112e-17 rpy=-7.9111e-17 -1.61837e-16 1.5708
- joint fastened_24_0: origin xyz=0 0.004 -0.01 rpy=-1.35122e-16 -1.0967e-16 1.5708 -> xyz=-2.77556e-17 0.004 -0.01 rpy=-1.62115e-16 -1.33819e-16 1.5708
- joint fastened_25_0: origin xyz=-0.01 0.004 1.38778e-17 rpy=-2.79844e-16 -8.78588e-17 1.5708 -> xyz=-0.01 0.004 -2.77556e-17 rpy=-2.75873e-15 -1.50918e-15 1.5708
- joint fastened_26_0: origin xyz=0 0.004 0.01 rpy=1.5708 -2.83107e-15 1.5708 -> xyz=-2.77556e-17 0.004 0.01 rpy=1.5708 -6.05072e-15 1.5708
- joint fastened_27_0: axis 0 1 0 -> 0 -1 0; origin xyz=-0.005 -0.019 -0.001488 rpy=0 -1.5708 4.71239 -> xyz=-0.002 -0.019 -0.001488 rpy=0 -1.5708 4.71239
- joint fastened_28_0: child limit_switch_2 -> limit_switch_1; origin xyz=-0.0104652 -0.031 0.031735 rpy=-8.33744e-18 -3.92985e-17 2.77556e-17 -> xyz=-0.0359195 -0.0632203 0.02135 rpy=0 -0 6.16298e-33; parent robot_belt_arm_endstop___mymod -> robot_belt_arm_socket_v2
- joint fastened_5_0: origin xyz=-2.77556e-17 0.0065 4.16334e-17 rpy=0 -1.5708 6.16777e-16 -> xyz=2.77556e-17 0.0065 2.77556e-17 rpy=0 -1.5708 1.39786e-15
- joint fastened_6_0: origin xyz=0.021 0.023 0.0345 rpy=3.14159 1.11575e-15 6.10623e-15 -> xyz=0.021 0.023 0.0345 rpy=3.14159 1.11575e-15 -5.4956e-15
- joint fastened_7_0: origin xyz=-0.0225 0.023 0.0385 rpy=-3.98519e-16 -2.34135e-17 -3.38618e-15 -> xyz=-0.0225 0.023 0.0385 rpy=-3.98519e-16 -2.34146e-17 3.35842e-15
- joint fastened_8_0: origin xyz=0.0269997 0.00750003 -0.00700002 rpy=0 -1.5708 3.14159 -> xyz=0.0119997 0.022 -0.027 rpy=0 -1.5708 3.14159
- joint fastened_9_0: origin xyz=0.0175 0.0008 0 rpy=-3.14159 4.0268e-16 -1.5708 -> xyz=0.0175 0.0008 -1.11022e-16 rpy=-3.14159 2.50042e-15 -1.5708
- joint final_motor_fastened_joint_0: origin xyz=0.199541 -0.0467529 -0.195348 rpy=7.61356e-15 3.49877e-15 -3.14159 -> xyz=0.199541 -0.0467529 -0.195348 rpy=7.61352e-15 3.4988e-15 -3.14159
- joint final_motor_fastened_joint_1: origin xyz=-0.145292 0.0466209 -0.195348 rpy=-2.52509e-16 5.33644e-16 -5.55126e-17 -> xyz=-0.145292 0.0466209 -0.195348 rpy=-2.52468e-16 5.33604e-16 -3.33068e-16
- joint final_motor_fastened_joint_2: origin xyz=-0.00527287 0.0177687 9.9951e-13 rpy=-1.01871e-15 -6.12848e-16 -0.0134012 -> xyz=-0.00527287 0.0177687 9.99485e-13 rpy=-1.01868e-15 -6.1282e-16 -0.0134012
- joint final_motor_fastened_joint_3: origin xyz=0.175273 -0.041981 0.204848 rpy=1.5708 -4.16334e-16 -0.348517 -> xyz=0.175273 -0.041981 0.204848 rpy=1.5708 2.77556e-17 -0.348517
- joint final_motor_fastened_joint_4: origin xyz=-0.34748 -0.0935381 -8.32667e-16 rpy=1.586e-15 -6.62775e-15 -3.14159 -> xyz=-0.34748 -0.0935381 -8.60423e-16 rpy=1.58602e-15 -6.62772e-15 -3.14159
- joint final_motor_fastened_joint_5: origin xyz=0.350607 -0.0217646 0.189648 rpy=7.06873e-16 -5.31245e-14 -0.123995 -> xyz=0.350607 -0.0217646 0.189648 rpy=7.06858e-16 -5.31245e-14 -0.123995
- joint final_motor_fastened_joint_7: origin xyz=-0.20806 0.129344 -0.189148 rpy=-9.77073e-15 1.25527e-15 -1.09828 -> xyz=-0.20806 0.129344 -0.189148 rpy=-9.77076e-15 1.25539e-15 -1.09828
- joint revolute_10_0: origin xyz=3.8384e-08 0.0135 0.064 rpy=3.14159 0.206001 2.87083e-15 -> xyz=3.8384e-08 0.0135 0.064 rpy=3.14159 0.232182 -1.3986e-15
- joint revolute_11_0: origin xyz=5.55112e-17 -1.38778e-17 -2.77556e-17 rpy=-3.14159 -1.40802 -3.09284e-14 -> xyz=2.60209e-18 -1.38778e-17 -2.77556e-17 rpy=-3.14159 -0.908726 -1.13289e-14
- joint revolute_12_0: origin xyz=-0.035954 -0.008 -0.0175303 rpy=1.5708 0.209788 6.52688e-16 -> xyz=-0.035954 -0.008 -0.0175303 rpy=1.5708 0.987621 -1.93546e-14
- joint revolute_13_0: origin xyz=-0.102411 1.16229e-09 0.0954576 rpy=-3.14159 -1.44881 3.14159 -> xyz=-0.102411 -2.58759e-08 0.0954575 rpy=-3.14159 -1.14393 3.14159
- joint revolute_14_0: origin xyz=0.102411 0.00500004 -0.0954576 rpy=1.5708 -1.12688e-14 1.5708 -> xyz=0.102411 0.00500004 -0.0954576 rpy=1.07158 -3.33067e-15 1.5708
- joint revolute_15_0: origin xyz=0.045 0.0035 0.008 rpy=4.88698e-16 1.23027 3.14159 -> xyz=0.045 0.0035 0.008 rpy=3.14159 1.43826 -1.14751e-14
- joint revolute_16_0: origin xyz=-0.139911 0.0205 -0.005 rpy=-1.5708 -1.31772 -2.26142e-14 -> xyz=-0.139911 0.0205 -0.005 rpy=1.5708 -1.04593 3.14159
- joint revolute_18_0: origin xyz=-0.102411 -1.11022e-16 0.0954576 rpy=3.14159 -1.44881 -3.14159 -> xyz=-0.102411 4.85723e-17 0.0954576 rpy=-3.14159 -1.14393 3.14159
- joint revolute_19_0: origin xyz=0.045 -0.0035 0.008 rpy=0 1.23027 -3.14159 -> xyz=0.045 -0.0035 0.008 rpy=-3.14159 1.43826 0
- joint revolute_1_0: origin xyz=-2.08167e-17 -0.0336603 0.0257 rpy=1.90568e-16 1.59644e-16 -1.27729 -> xyz=4.85723e-17 -0.0336603 0.0257 rpy=2.02624e-16 -4.55524e-17 0.559643
- joint revolute_22_0: origin xyz=0.0269997 0.00750003 -0.001 rpy=1.93138e-15 -4.34816e-16 2.80332e-15 -> xyz=0.0119997 0.022 -0.021 rpy=1.94752e-15 -1.28355e-15 9.71452e-16
- joint revolute_24_0: origin xyz=0.03 0.0089 -0.012 rpy=-0.377454 4.77396e-15 -1.5708 -> xyz=0.03 0.0089 -0.012 rpy=-0.377448 2.52576e-15 -1.5708
- joint revolute_25_0: origin xyz=-0.11402 0.0812835 0.001 rpy=0 1.5708 -3.56578e-06 -> xyz=-0.11402 0.0812835 0.001 rpy=0 1.5708 0.311198
- joint revolute_26_0: origin xyz=-5.55112e-17 0.00500004 -1.04083e-17 rpy=-1.5708 -2.22045e-16 1.5708 -> xyz=5.55112e-17 0.00500004 5.55112e-17 rpy=-2.07001 1.11022e-16 1.5708
- joint revolute_27_0: origin xyz=0 -0.00500004 -1.38778e-17 rpy=1.5708 4.996e-16 -1.5708 -> xyz=5.55112e-17 -0.00500004 0 rpy=2.2706 -4.32987e-15 -1.5708
- joint revolute_28_0: origin xyz=-0.102411 0.00500004 0.0954576 rpy=-1.84603 -5.55112e-17 1.5708 -> xyz=-0.102411 0.00500004 0.0954576 rpy=-2.15739 -3.60822e-15 1.5708
- joint revolute_29_0: origin xyz=-0.102411 -0.00500004 0.0954576 rpy=1.84603 -4.4964e-15 -1.5708 -> xyz=-0.102411 -0.00500004 0.0954576 rpy=2.15739 6.10623e-16 -1.5708
- joint revolute_2_0: origin xyz=3.81639e-17 1.38778e-17 0 rpy=-1.87643e-15 1.85486e-16 2.84045 -> xyz=5.55112e-17 1.73472e-16 3.33067e-16 rpy=-2.08079e-15 3.12771e-16 1.00352
- joint revolute_30_0: origin xyz=3.8384e-08 0.026 0.064 rpy=-1.5708 5.88418e-15 5.85208e-15 -> xyz=3.8384e-08 0.026 0.064 rpy=-1.5708 -1.44676e-15 6.57373e-15
- joint revolute_31_0: origin xyz=-0.03 0.026 0.076 rpy=-3.14159 1.44879 -3.14159 -> xyz=-0.03 0.026 0.076 rpy=-3.14159 1.14391 -3.14159
- joint revolute_32_0: origin xyz=-0.03 -0.026 0.076 rpy=-3.14159 1.44879 -3.14159 -> xyz=-0.03 -0.026 0.076 rpy=-3.14159 1.14391 -3.14159
- joint revolute_3_0: origin xyz=-5.55112e-17 -0.00500004 1.38778e-17 rpy=1.84603 -5.05151e-15 -1.5708 -> xyz=2.77556e-17 -0.00500004 4.16334e-17 rpy=2.15739 -4.44089e-16 -1.5708
- joint revolute_4_0: origin xyz=2.77556e-17 0.00500004 4.16334e-17 rpy=-1.84603 7.21645e-16 1.5708 -> xyz=-5.55112e-17 0.00500004 -4.16334e-17 rpy=-2.15739 -4.88498e-15 1.5708
- joint revolute_5_0: origin xyz=-2.77556e-17 -0.007 0 rpy=-8.87308e-07 1.56423e-15 1.5708 -> xyz=-0.015 0.0075 -0.02 rpy=3.32548e-07 1.99214e-15 1.5708
- joint revolute_6_0: origin xyz=-1.94289e-16 5.55112e-17 0.005 rpy=0 -1.5708 3.14159 -> xyz=-5.55112e-17 8.32667e-17 0.005 rpy=0 -1.5708 3.45279
- joint revolute_8_0: origin xyz=0.102411 -0.00500004 -0.0954576 rpy=-1.09686 -1.52101e-14 -1.5708 -> xyz=0.102411 -0.00500004 -0.0954576 rpy=-0.397052 -1.6348e-14 -1.5708
- joint revolute_9_0: origin xyz=-4.83882e-08 -0.02 0.064 rpy=-3.14159 -0.908 3.14159 -> xyz=3.53185e-08 -0.02 0.064 rpy=3.14159 -1.21288 -3.14159
