Commit message: feat: Rename revolutes for undestandable names

File: src/robots/community_robot_arm/urdf/processed/community_robot_arm_with_collisions.urdf (robot description, URDF)
Before this commit: robot complete_robotic_arm_assembly_with_dual_manipulator_140mm_shank, 102 links, 101 joints
Joints:
- removed joint revolute_10_0
- removed joint revolute_1_0
- removed joint revolute_9_0
- added joint base_yaw_joint: type continuous, parent robot_belt_arm_socket_v2, child robot_belt_arm_main_body_v2______mymod, origin xyz=4.85723e-17 -0.0336603 0.0257 rpy=2.02624e-16 -4.55524e-17 0.559643, axis 0 0 -1
- added joint elbow_pitch_joint: type continuous, parent robot_belt_arm_main_body_v2______mymod, child robot_belt_arm_gear_body, origin xyz=3.8384e-08 0.0135 0.064 rpy=3.14159 0.232182 -1.3986e-15, axis 0 1 0
- added joint shoulder_pitch_joint: type continuous, parent robot_belt_arm_main_body_v2______mymod, child robot_belt_arm_gear_body_1, origin xyz=3.53175e-08 -0.02 0.064 rpy=3.14159 -1.21288 -3.14159, axis 0 1 0

File: src/robots/community_robot_arm/urdf/raw/community_robot_arm_full.urdf (robot description, URDF)
Before this commit: robot complete_robotic_arm_assembly_with_dual_manipulator_140mm_shank, 105 links, 104 joints
Joints:
- removed joint revolute_10_0
- removed joint revolute_1_0
- removed joint revolute_9_0
- added joint base_yaw_joint: type continuous, parent robot_belt_arm_socket_v2, child robot_belt_arm_main_body_v2______mymod, origin xyz=4.85723e-17 -0.0336603 0.0257 rpy=2.02624e-16 -4.55524e-17 0.559643, axis 0 0 -1
- added joint elbow_pitch_joint: type continuous, parent robot_belt_arm_main_body_v2______mymod, child robot_belt_arm_gear_body, origin xyz=3.8384e-08 0.0135 0.064 rpy=3.14159 0.232182 -1.3986e-15, axis 0 1 0
- added joint shoulder_pitch_joint: type continuous, parent robot_belt_arm_main_body_v2______mymod, child robot_belt_arm_gear_body_1, origin xyz=3.53175e-08 -0.02 0.064 rpy=3.14159 -1.21288 -3.14159, axis 0 1 0

File: src/robots/community_robot_arm/urdf/raw/community_robot_arm_slim.urdf (robot description, URDF)
Before this commit: robot complete_robotic_arm_assembly_with_dual_manipulator_140mm_shank, 102 links, 101 joints
Joints:
- removed joint revolute_10_0
- removed joint revolute_1_0
- removed joint revolute_9_0
- added joint base_yaw_joint: type continuous, parent robot_belt_arm_socket_v2, child robot_belt_arm_main_body_v2______mymod, origin xyz=4.85723e-17 -0.0336603 0.0257 rpy=2.02624e-16 -4.55524e-17 0.559643, axis 0 0 -1
- added joint elbow_pitch_joint: type continuous, parent robot_belt_arm_main_body_v2______mymod, child robot_belt_arm_gear_body, origin xyz=3.8384e-08 0.0135 0.064 rpy=3.14159 0.232182 -1.3986e-15, axis 0 1 0
- added joint shoulder_pitch_joint: type continuous, parent robot_belt_arm_main_body_v2______mymod, child robot_belt_arm_gear_body_1, origin xyz=3.53175e-08 -0.02 0.064 rpy=3.14159 -1.21288 -3.14159, axis 0 1 0

File: src/robots/community_robot_arm/urdf/spherized/community_robot_arm_slim_spherized.urdf (robot description, URDF)
Before this commit: robot complete_robotic_arm_assembly_with_dual_manipulator_140mm_shank, 102 links, 101 joints
Joints:
- removed joint revolute_10_0
- removed joint revolute_1_0
- removed joint revolute_9_0
- added joint base_yaw_joint: type continuous, parent robot_belt_arm_socket_v2, child robot_belt_arm_main_body_v2______mymod, origin xyz=4.85723e-17 -0.0336603 0.0257 rpy=2.02624e-16 -4.55524e-17 0.559643, axis 0 0 -1
- added joint elbow_pitch_joint: type continuous, parent robot_belt_arm_main_body_v2______mymod, child robot_belt_arm_gear_body, origin xyz=3.8384e-08 0.0135 0.064 rpy=3.14159 0.232182 -1.3986e-15, axis 0 1 0
- added joint shoulder_pitch_joint: type continuous, parent robot_belt_arm_main_body_v2______mymod, child robot_belt_arm_gear_body_1, origin xyz=3.53175e-08 -0.02 0.064 rpy=3.14159 -1.21288 -3.14159, axis 0 1 0
