Commit message: feat: solver with rust and also new obstacles

File: src/robots/community_robot_arm/urdf/raw/obstacles/box_obstacle.urdf (robot description, URDF)
Before this commit: robot box_obstacle, 2 links, 1 joints
Joints:
- joint obstacle_box_joint: origin xyz=0.3 0.15 0.2 rpy=0 0 0 -> xyz=0.3 0.0 0.15 rpy=0 0 0

File: src/robots/community_robot_arm/urdf/spherized/obstacles/box_obstacle_spherized.urdf (robot description, URDF)
Before this commit: robot box_obstacle, 2 links, 1 joints
Links:
- link obstacle_box_link: geometry collision sphere radius=0.12889; collision sphere radius=0.129903
Joints:
- joint obstacle_box_joint: origin xyz=0.3 0.15 0.2 rpy=0 0 0 -> xyz=0.3 0.0 0.15 rpy=0 0 0
